File: PCB/analog_SWR_detection/analog_SWR_detection_version2/analog_SWR_detection_version2.sch (KiCad schematic (older format))
At the start: 36 parts, among them J1 Conn_Coaxial, J2 Conn_01x04_Male, J3 Screw_Terminal_01x02, J4 Screw_Terminal_01x02, J5 Screw_Terminal_01x02, J6 Screw_Terminal_01x02, J7 Conn_Coaxial, U1 LM358N, U2 LM358N, U3 LM358

Commit message: update on circuit board
Parts:
- removed J1, J7: Conn_Coaxial, Connector_Coaxial:BNC_Amphenol_B6252HB-NPP3G-50_Horizontal, symbol Connector:Conn_Coaxial
- removed J2: Conn_01x04_Male, symbol Connector:Conn_01x04_Male
- added J6: Screw_Terminal_01x02, symbol Connector:Screw_Terminal_01x02
- U3: footprint (none) -> Package_DIP:DIP-8_W7.62mm_Socket
- gave numbers to parts that had none: 8
- renumbered C6 to C5, C7 to C6, C5 to C8, J3 to J2, J4 to J3, J5 to J4, J6 to J5, R12 to R6, R14 to R8, U3 to U2, U2 to U4, U3 to U4
Connections:
- net GND: now also J1.3, J3.1 (Pin_1); no longer J2.1 (Pin_1)
- net at R3.1, RV1.5, U1.1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: now also J1.6, J4.2 (Pin_2); no longer J2.2 (Pin_2)
- net at C1.1: now also J1.4, J3.2 (Pin_2)
- net at C4.2, U1.6 (-), U1.7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: now also J1.7, J5.1 (Pin_1); no longer J3.1 (Pin_1)
- net at U1.4 (V-), U2.4 (V-), U3.4 (V-): now also J1.2, J2.2 (Pin_2)
- net at U1.8 (V+), U2.8 (V+), U3.8 (V+): now also J1.1, J2.1 (Pin_1)
- net at C8.1, R11.2, R6.1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: now also J1.8, J1.9, J6.1 (Pin_1), J6.2 (Pin_2)
- net at R7.1, RV3.2, U2.1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: now also J5.2 (Pin_2); no longer J3.2 (Pin_2)
- net at C6.2, U2.6 (-), U2.7: now also J1.5, J4.1 (Pin_1)
Other:
- note added: "Input"
- note added: "What is in each pin of the screw terminal:\nFrom left to right\n1 - poisitve source\n2 - negative source\n3 - ground\n4 - signal input for the circuit\n5 - signal output of the whole ircuit\n6 - output of first high pass part\n7 - output of low pass part\n8 - output of amplification part\n9 - output of retification part\n10 - output of envelope part"
- note added: "What is in each pin on DB9\n1 - positive source\n2 - negative source\n3 - ground\n4 - signal input for the circuit\n5 - signal output of the whole circuit\n6 - output of first high pass part\n7 - output of low pass part\n8 - output of retification\n9 - output of envelope"
- note removed: "This should input arduino voltage"
- moved on the sheet: J1, J2, J3, J4, J5
